File: cherrycam/cherrycam.kicad_pcb (KiCad board)
At the start: 4 copper layers, 100 x 70 mm, 51 parts, among them J1 DF40C-100DS-0.4V_51_, J2 DF40C-100DS-0.4V_51_, J3 Conn_01x22, J4 Conn_01x08, J5 Micro_SD_Card_Det1, J6 Conn_01x04, J7 USB_C_Receptacle_USB2.0_16P, Q1 BSS138, SW1 SW_Push, U1 USBLC6-2SC6, U2 AP2112K-3.3, U3 AP2112K-1.8, U4 MIC5504-2.8YM5, U5 W25Q128JVS

Commit message: work on pcb + journal entry
Parts:
- added REF**: MountingHole_3.2mm_M3_ISO7380_Pad, MountingHole:MountingHole_3.2mm_M3_ISO7380_Pad, F.Cu at (4.00, 66.0)
- added REF**: MountingHole_3.2mm_M3_ISO7380_Pad, MountingHole:MountingHole_3.2mm_M3_ISO7380_Pad, F.Cu at (96.0, 4.00)
- added REF**: MountingHole_3.2mm_M3_ISO7380_Pad, MountingHole:MountingHole_3.2mm_M3_ISO7380_Pad, F.Cu at (4.00, 4.00)
- added REF**: MountingHole_3.2mm_M3_ISO7380_Pad, MountingHole:MountingHole_3.2mm_M3_ISO7380_Pad, F.Cu at (96.0, 66.0)
- moved R4 85.1 mm to (39.5, 2.00), turned to 180 degrees
- moved C_CAM4 79.9 mm to (46.5, 10.5)
- moved R3 79.2 mm to (39.5, 6.00)
- moved J4 78.7 mm to (96.5, 26.8)
- moved C_CAM3 78.2 mm to (40.5, 10.5)
- moved C1 77.1 mm to (5.14, 57.5), turned to 90 degrees
- moved SW1 77.0 mm to (82.0, 4.75)
- moved C_CAM2 76.9 mm to (34.5, 10.5)
- moved C_CAM1 76.2 mm to (28.5, 10.5)
- moved J3 75.3 mm to (50.0, 2.90), turned to 180 degrees
- moved D2 71.4 mm to (88.4, 3.81)
- moved U2 69.7 mm to (10.0, 58.0)
- moved J1 67.7 mm to (38.0, 22.5)
- moved Q1 67.4 mm to (89.5, 30.5), turned to 180 degrees
- moved C2 67.4 mm to (14.6, 57.5), turned to 90 degrees
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Routing:
- added copper zone on In2.Cu, net +3V3
- added copper zone on In1.Cu, net GND

Commit message: new update
Parts:
- moved J5 65.0 mm to (13.6, 37.9), turned to -90 degrees
- moved R13 44.1 mm to (33.0, 40.5), turned to -90 degrees
- moved C12 42.4 mm to (33.0, 44.6), turned to 90 degrees
- moved R12 41.0 mm to (33.0, 37.5), turned to -90 degrees
- moved R11 38.0 mm to (33.0, 34.5), turned to -90 degrees
- moved R10 35.3 mm to (33.0, 31.5), turned to -90 degrees
- moved R9 32.9 mm to (33.0, 28.5), turned to -90 degrees
- moved R8 22.5 mm to (38.0, 17.9), turned to 180 degrees
- moved R7 22.4 mm to (38.0, 14.4), turned to 180 degrees
- moved C1 21.9 mm to (27.0, 59.6)
- moved C4 21.9 mm to (43.5, 59.5)
- moved C8 21.9 mm to (70.0, 59.5)
- moved C9 21.9 mm to (73.5, 59.5)
- moved U2 21.9 mm to (31.8, 60.0)
- moved U4 21.9 mm to (65.5, 60.0)
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- renumbered REF** to REF1, REF** to REF2, REF** to REF3, REF** to REF5
Connections:
- net /compute/CM4_1V8_OUT renamed CM4_1V8_OUT
- net /compute/CM4_3V3_OUT renamed CM4_3V3_OUT
- net /compute/DISP_MISO renamed DISP_MISO
- net /compute/SD_PWR_ON renamed SD_PWR_ON
- net /compute/USB_N renamed USB_N
- net /compute/USB_P renamed USB_P
- net /display/DISP_BL renamed DISP_BL
- net /power/+2V8 renamed +2V8
- net /storage_ui/SD_CD renamed SD_CD
- C1 pad 2: /power/5V_MAIN -> 5V_MAIN
- C10 pad 1: /power/5V_MAIN -> 5V_MAIN
- C11 pad 1: /power/5V_MAIN -> 5V_MAIN
- C12 pad 1: /storage_ui/+3V3 -> +3V3
- C13 pad 1: /storage_ui/+3V3 -> +3V3
- C14 pad 1: /storage_ui/+3V3 -> +3V3
- C15 pad 1: /storage_ui/SHUTTER -> SHUTTER
- C_CAM1 pad 1: /sensor/+3V3 -> +3V3
- C_CAM2 pad 1: /sensor/+3V3 -> +3V3
- C_CAM3 pad 1: /sensor/+1V8 -> +1V8
- C_CAM4 pad 1: /sensor/+1V8 -> +1V8
- F1 pad 2: /power/5V_MAIN -> 5V_MAIN
- J1 pad 21: /compute/LED_ACT -> LED_ACT
- J1 pad 24: /compute/DISP_DC -> DISP_DC
- J1 pad 25: /compute/DISP_RST -> DISP_RST
- J1 pad 26: /compute/QSPI_MISO -> QSPI_MISO
- J1 pad 27: /compute/QSPI_MOSI -> QSPI_MOSI
- J1 pad 28: /compute/SHUTTER -> SHUTTER
- J1 pad 37: /compute/DISP_CS -> DISP_CS
- J1 pad 38: /compute/DISP_CLK -> DISP_CLK
- J1 pad 44: /compute/DISP_MOSI -> DISP_MOSI
- J1 pad 49: /compute/QSPI_CLK -> QSPI_CLK
- J1 pad 50: /compute/QSPI_CS -> QSPI_CS
- J1 pad 51: /compute/UART_TX -> UART_TX
- J1 pad 55: /compute/UART_RX -> UART_RX
- J1 pad 57: /compute/SD_CLK -> SD_CLK
- J1 pad 61: /compute/SD_DAT3 -> SD_DAT3
- J1 pad 62: /compute/SD_CMD -> SD_CMD
- J1 pad 63: /compute/SD_DAT0 -> SD_DAT0
- J1 pad 67: /compute/SD_DAT1 -> SD_DAT1
- J1 pad 69: /compute/SD_DAT2 -> SD_DAT2
- J1 pad 77: /compute/5V_MAIN -> 5V_MAIN
- J1 pad 79: /compute/5V_MAIN -> 5V_MAIN
- J1 pad 80: /compute/CAM_SCL -> CAM_SCL
- J1 pad 81: /compute/5V_MAIN -> 5V_MAIN
- J1 pad 82: /compute/CAM_SDA -> CAM_SDA
- J1 pad 83: /compute/5V_MAIN -> 5V_MAIN
- J1 pad 85: /compute/5V_MAIN -> 5V_MAIN
- J1 pad 87: /compute/5V_MAIN -> 5V_MAIN
- J1 pad 99: /compute/5V_MAIN -> 5V_MAIN
- J2 pad 15: /compute/CAM1_D0_N -> CAM1_D0_N
- J2 pad 17: /compute/CAM1_D0_P -> CAM1_D0_P
- J2 pad 21: /compute/CAM1_D1_N -> CAM1_D1_N
- J2 pad 23: /compute/CAM1_D1_P -> CAM1_D1_P
- J2 pad 27: /compute/CAM1_C_N -> CAM1_C_N
- J2 pad 29: /compute/CAM1_C_P -> CAM1_C_P
- J2 pad 33: /compute/CAM1_D2_N -> CAM1_D2_N
- J2 pad 35: /compute/CAM1_D2_P -> CAM1_D2_P
- J2 pad 39: /compute/CAM1_D3_N -> CAM1_D3_N
- J2 pad 41: /compute/CAM1_D3_P -> CAM1_D3_P
- J2 pad 97: /compute/CAM_GPIO -> CAM_GPIO
- J3 pad 11: /sensor/CAM1_D2_N -> CAM1_D2_N
- J3 pad 12: /sensor/CAM1_D2_P -> CAM1_D2_P
- J3 pad 14: /sensor/CAM1_D3_N -> CAM1_D3_N
- J3 pad 15: /sensor/CAM1_D3_P -> CAM1_D3_P
- J3 pad 17: /sensor/CAM_SCL -> CAM_SCL
- J3 pad 18: /sensor/CAM_SDA -> CAM_SDA
- J3 pad 2: /sensor/CAM1_D0_N -> CAM1_D0_N
- J3 pad 20: /sensor/CAM_GPIO -> CAM_GPIO
- J3 pad 21: /sensor/+3V3 -> +3V3
- J3 pad 22: /sensor/+3V3 -> +3V3
- J3 pad 3: /sensor/CAM1_D0_P -> CAM1_D0_P
- J3 pad 5: /sensor/CAM1_D1_N -> CAM1_D1_N
- J3 pad 6: /sensor/CAM1_D1_P -> CAM1_D1_P
- J3 pad 8: /sensor/CAM1_C_N -> CAM1_C_N
- J3 pad 9: /sensor/CAM1_C_P -> CAM1_C_P
- J4 pad 1: /display/+3V3 -> +3V3
- J4 pad 3: /display/DISP_CS -> DISP_CS
- J4 pad 4: /display/DISP_RST -> DISP_RST
- J4 pad 5: /display/DISP_DC -> DISP_DC
- J4 pad 6: /display/DISP_MOSI -> DISP_MOSI
- J4 pad 7: /display/DISP_CLK -> DISP_CLK
- J5 pad 1: /storage_ui/SD_DAT2 -> SD_DAT2
- J5 pad 2: /storage_ui/SD_DAT3 -> SD_DAT3
- J5 pad 4: /storage_ui/+3V3 -> +3V3
- J5 pad 7: /storage_ui/SD_DAT0 -> SD_DAT0
- J5 pad 8: /storage_ui/SD_DAT1 -> SD_DAT1
- J6 pad 2: /storage_ui/+3V3 -> +3V3
- J6 pad 3: /storage_ui/UART_TX -> UART_TX
- J6 pad 4: /storage_ui/UART_RX -> UART_RX
- R10 pad 1: /storage_ui/+3V3 -> +3V3
- R10 pad 2: /storage_ui/SD_DAT2 -> SD_DAT2
- R11 pad 1: /storage_ui/SD_DAT3 -> SD_DAT3
- R11 pad 2: /storage_ui/+3V3 -> +3V3
- R12 pad 1: /storage_ui/+3V3 -> +3V3
- R13 pad 1: /storage_ui/+3V3 -> +3V3
- R13 pad 2: /storage_ui/SHUTTER -> SHUTTER
- R14 pad 1: /storage_ui/+3V3 -> +3V3
- R15 pad 1: /storage_ui/LED_ACT -> LED_ACT
- R3 pad 1: /sensor/+3V3 -> +3V3
- R3 pad 2: /sensor/CAM_SCL -> CAM_SCL
- R4 pad 1: /sensor/CAM_SDA -> CAM_SDA
- R4 pad 2: /sensor/+3V3 -> +3V3
- R5 pad 1: /storage_ui/SD_CLK -> SD_CLK
- R6 pad 1: /storage_ui/SD_CMD -> SD_CMD
- R7 pad 1: /storage_ui/+3V3 -> +3V3
- R7 pad 2: /storage_ui/SD_CMD -> SD_CMD
- R8 pad 1: /storage_ui/+3V3 -> +3V3
- R8 pad 2: /storage_ui/SD_DAT0 -> SD_DAT0
- R9 pad 1: /storage_ui/+3V3 -> +3V3
- R9 pad 2: /storage_ui/SD_DAT1 -> SD_DAT1
- SW1 pad 1: /storage_ui/SHUTTER -> SHUTTER
- U1 pad 5: /power/5V_MAIN -> 5V_MAIN
- U2 pad 1: /power/5V_MAIN -> 5V_MAIN
- U2 pad 3: /power/5V_MAIN -> 5V_MAIN
- U5 pad 1: /storage_ui/QSPI_CS -> QSPI_CS
- U5 pad 2: /storage_ui/QSPI_MISO -> QSPI_MISO
- U5 pad 3: /storage_ui/+3V3 -> +3V3
- U5 pad 5: /storage_ui/QSPI_MOSI -> QSPI_MOSI
- U5 pad 6: /storage_ui/QSPI_CLK -> QSPI_CLK
- U5 pad 7: /storage_ui/+3V3 -> +3V3
- U5 pad 8: /storage_ui/+3V3 -> +3V3
Routing:
- removed copper zone on In2.Cu, net +3V3
- removed copper zone on In1.Cu, net GND

Commit message: im going through changesss
Parts:
- moved C_CAM1 56.9 mm to (41.0, 66.0)
- moved C_CAM2 56.9 mm to (47.1, 66.0)
- moved C_CAM3 56.9 mm to (53.0, 66.0)
- moved C_CAM4 56.9 mm to (59.0, 66.0)
- moved R5 35.4 mm to (33.0, 48.0)
- moved R6 35.4 mm to (33.0, 52.0)
- moved Q1 27.5 mm to (87.0, 60.4)
- moved J1 24.4 mm to (50.0, 50.0), turned to 180 degrees
- moved J6 22.1 mm to (96.5, 28.9)
- moved J2 21.6 mm to (50.0, 27.0), turned to 180 degrees
- moved J4 15.3 mm to (96.5, 42.1)
- moved C10 7.48 mm to (76.0, 26.0)
- moved C11 7.48 mm to (72.5, 26.0)
- moved R1 6.80 mm to (83.0, 30.5)
- moved R2 6.80 mm to (83.0, 33.5)
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