File: cherrycam/sheets/display.kicad_sch (KiCad schematic)
At the start: 0 parts

Commit message: massive updates + 30 june journal entry
Parts:
- added J4: Conn_01x08, symbol Connector_Generic:Conn_01x08
- added Q1: BSS138, Package_TO_SOT_SMD:SOT-23, symbol Transistor_FET:BSS138
Connections:
- new net: J4.8 (Pin_8), Q1.3 (D)
- new net +3V3: J4.1 (Pin_1)
- new net DISP_BL: Q1.1 (G)
- new net DISP_CLK: J4.7 (Pin_7)
- new net DISP_CS: J4.3 (Pin_3)
- new net DISP_DC: J4.5 (Pin_5)
- new net DISP_MOSI: J4.6 (Pin_6)
- new net DISP_RST: J4.4 (Pin_4)
- new net GND: J4.2 (Pin_2), Q1.2 (S)
