File: cherrycam/sheets/sensor.kicad_sch (KiCad schematic)
At the start: 0 parts

Commit message: massive updates + 30 june journal entry
Parts:
- added C_CAM1, C_CAM3: 100nF, symbol Device:C
- added C_CAM2, C_CAM4: 10µF, symbol Device:C
- added J3: Conn_01x22, Connector_FFC-FPC:Hirose_FH12-22S-0.5SH_1x22-1MP_P0.50mm_Horizontal, symbol Connector_Generic:Conn_01x22
- added R3, R4: 4.7k, symbol Device:R
Connections:
- new net +1V8: C_CAM3.1, C_CAM4.1
- new net +3V3: C_CAM1.1, C_CAM2.1, J3.21 (Pin_21), J3.22 (Pin_22), R3.1, R4.2
- new net CAM1_C_N: J3.8 (Pin_8)
- new net CAM1_C_P: J3.9 (Pin_9)
- new net CAM1_D0_N: J3.2 (Pin_2)
- new net CAM1_D0_P: J3.3 (Pin_3)
- new net CAM1_D1_N: J3.5 (Pin_5)
- new net CAM1_D1_P: J3.6 (Pin_6)
- new net CAM1_D2_N: J3.11 (Pin_11)
- new net CAM1_D2_P: J3.12 (Pin_12)
- new net CAM1_D3_N: J3.14 (Pin_14)
- new net CAM1_D3_P: J3.15 (Pin_15)
- new net CAM_GPIO: J3.20 (Pin_20)
- new net CAM_SCL: J3.17 (Pin_17), R3.2
- new net CAM_SDA: J3.18 (Pin_18), R4.1
- new net GND: C_CAM1.2, C_CAM2.2, C_CAM3.2, C_CAM4.2, J3.1 (Pin_1), J3.10 (Pin_10), J3.13 (Pin_13), J3.16 (Pin_16), J3.19 (Pin_19), J3.4 (Pin_4), J3.7 (Pin_7)
