File: cherrycam/sheets/storage_ui.kicad_sch (KiCad schematic)
At the start: 0 parts

Commit message: massive updates + 30 june journal entry
Parts:
- added C12, C13, C15: 100nF, symbol Device:C
- added C14: 10µF, symbol Device:C
- added D1, D2: LED, symbol Device:LED
- added J5: Micro_SD_Card_Det1, symbol Connector:Micro_SD_Card_Det1
- added J6: Conn_01x04, symbol Connector_Generic:Conn_01x04
- added R10, R11, R12, R7, R8, R9: R, symbol Device:R
- added R13: 10kΩ, symbol Device:R
- added R14, R15: 330Ω, symbol Device:R
- added R5, R6: 47Ω, symbol Device:R
- added SW1: SW_Push, symbol Switch:SW_Push
- added U5: W25Q128JVS, Package_SO:SOIC-8_5.3x5.3mm_P1.27mm, symbol Memory_Flash:W25Q128JVS
Connections:
- new net: D2.2 (A), R15.2
- new net: D1.2 (A), R14.2
- new net: J5.3 (CMD), R6.2
- new net: J5.5 (CLK), R5.2
- new net +3V3: C12.1, C13.1, C14.1, J5.4 (VDD), J6.2 (Pin_2), R10.1, R11.2, R12.1, R13.1, R14.1, R7.1, R8.1, R9.1, U5.3 (~{WP}/IO_{2}), U5.7 (~{HOLD}/~{RESET}/IO_{3}), U5.8 (VCC)
- new net GND: C12.2, C13.2, C14.2, C15.2, D1.1 (K), D2.1 (K), J5.6 (VSS), J6.1 (Pin_1), SW1.2, U5.4 (GND)
- new net LED_ACT: R15.1
- new net QSPI_CLK: U5.6 (CLK)
- new net QSPI_CS: U5.1 (~{CS})
- new net QSPI_MISO: U5.2 (DO/IO_{1})
- new net QSPI_MOSI: U5.5 (DI/IO_{0})
- new net SD_CD: J5.9 (DET), R12.2
- new net SD_CLK: R5.1
- new net SD_CMD: R6.1, R7.2
- new net SD_DAT0: J5.7 (DAT0), R8.2
- new net SD_DAT1: J5.8 (DAT1), R9.2
- new net SD_DAT2: J5.1 (DAT2), R10.2
- new net SD_DAT3: J5.2 (DAT3/CD), R11.1
- new net SHUTTER: C15.1, R13.2, SW1.1
- new net UART_RX: J6.4 (Pin_4)
- new net UART_TX: J6.3 (Pin_3)
